File: PLC4UNI NIZAO/PLC4UNI NIZAO/EnergyMeter.kicad_sch (KiCad schematic)
At the start: 0 parts

Commit message: commit 4 Schematic
Parts:
- added C35, C36: 33NF, Capacitor_SMD_AKL:C_0603_1608Metric, symbol Capacitor_AKL:C_0603
- added C37: 68NF, Capacitor_SMD_AKL:C_0603_1608Metric, symbol Capacitor_AKL:C_0603
- added C38, C39, C40: 100NF, Capacitor_SMD_AKL:C_0603_1608Metric, symbol Capacitor_AKL:C_0603
- added R53, R54: 0.51, Resistor_SMD_AKL:R_0805_2012Metric, symbol Resistor_US_AKL:R_0805
- added R55, R56: 1K, Resistor_SMD_AKL:R_0603_1608Metric, symbol Resistor_US_AKL:R_0603
- added R57, R59, R60, R61, R62: 390K, Resistor_SMD_AKL:R_0603_1608Metric, symbol Resistor_US_AKL:R_0603
- added R58: 510, Resistor_SMD_AKL:R_0603_1608Metric, symbol Resistor_US_AKL:R_0603
- added R63, R64, R65, R66: 4.7K, Resistor_SMD_AKL:R_0603_1608Metric, symbol Resistor_US_AKL:R_0603
- added TP10, TP11, TP5, TP9: TestPoint_Hole1, 4ms_TestPoint:TestPoint_WireHole, symbol MG_ELECTROMECANICAL:TestPoint_Hole1
- added U16: BL0942, EasyEDA:SSOP-10_L4.9-W3.9-P1.00-LS6.0-BL, symbol EasyEDA:BL0942
- added U17: B0303S-1WR3_C7465185, EasyEDA:PWRM-TH_BXXXXS-1WR3, symbol EasyEDA:B0303S-1WR3_C7465185
- added U18: ISO7021DR, EasyEDA:SOIC-8_L4.9-W3.9-P1.27-LS6.0-BL, symbol EasyEDA:ISO7021DR
Connections:
- new net: C37.2, R58.2, R62.2, TP9.1, U16.4 (VP)
- new net: R59.2, R60.1
- new net: R60.2, R61.1
- new net: R63.1, U16.9 (RX/SDI), U18.6 (OUTB)
- new net: C36.1, R56.2, TP11.1, U16.3 (IN)
- new net: R64.1, U16.10 (TX/SDO), U18.7 (INA)
- new net: C35.2, R55.2, TP10.1, U16.2 (IP)
- new net: R57.2, R59.1
- new net: R61.2, R62.1
- new net +3.3V: C40.2, R65.2, R66.2, U17.2 (+Vin), U18.1 (VCC1)
- new net CT_N: R54.2, R56.1
- new net CT_P: R53.1, R55.1
- new net Earth: C35.1, C36.2, C37.1, C38.1, C39.1, R53.2, R54.1, R58.1, U16.5 (GND), U16.7 (SEL), U17.3 (-Vout), U18.5 (GND2)
- new net GND: C40.1, U17.1 (-Vin), U18.4 (GND1)
- new net RX: R65.1, U18.3 (INB)
- new net TX: R66.1, U18.2 (OUTA)
- new net VCC: C38.2, C39.2, R63.2, R64.2, TP5.1, U16.1 (VDD), U16.8 (SCLK_BPS), U17.4 (+Vout), U18.8 (VCC2)
- new net VIN_P: R57.1
