File: PLC4UNI NIZAO/PLC4UNI NIZAO/IN-DI.kicad_sch (KiCad schematic)
At the start: 5 parts

Commit message: commit 4 Schematic
Parts:
- removed C7: 2.2NF, PCM_SparkFun-Capacitor:C_0603_1608Metric, symbol PCM_SparkFun-Capacitor:C
- removed C8: 1NF, PCM_SparkFun-Capacitor:C_0603_1608Metric, symbol PCM_SparkFun-Capacitor:C
- removed R13: 3.6K, symbol Device:R_US
- removed R14: 3.3K, symbol Device:R_US
- removed R15: 22K, symbol Device:R_US
- added C18: 2.2NF, Capacitor_SMD_AKL:C_0603_1608Metric, symbol Capacitor_AKL:C_0603
- added C19: 1NF, Capacitor_SMD_AKL:C_0603_1608Metric, symbol Capacitor_AKL:C_0603
- added R28: 3.6K, Resistor_SMD_AKL:R_0603_1608Metric, symbol Resistor_US_AKL:R_0603
- added R29: 3.3K, Resistor_SMD_AKL:R_0603_1608Metric, symbol Resistor_US_AKL:R_0603
- added R30: 22K, Resistor_SMD_AKL:R_0603_1608Metric, symbol Resistor_US_AKL:R_0603
- added U3: AT3H4B-CUH-S, easyeda2kicad:SSOP-4_L2.7-W4.6-P1.27-LS7.0-TL, symbol easyeda2kicad:AT3H4B-CUH-S
Connections:
- net COM: now also C18.2, R29.1, U3.2
- net GND: now also C19.2, U3.3
- net IN: now also R28.1
- net OUT: now also C19.1, R30.1, U3.4
- new net: C18.1, R28.2, R29.2, U3.1
- new net +3.3V: R30.2
