File: PLC4UNI NIZAO/PLC4UNI NIZAO/TC.kicad_sch (KiCad schematic)
At the start: 0 parts

Commit message: commit 4 Schematic
Parts:
- added C27, C29, C30: 0.01UF, Capacitor_SMD_AKL:C_0603_1608Metric, symbol Capacitor_AKL:C_0603
- added C28, C31: 100NF, Capacitor_SMD_AKL:C_0603_1608Metric, symbol Capacitor_AKL:C_0603
- added R35, R36: 0R, Resistor_SMD_AKL:R_0603_1608Metric, symbol Resistor_US_AKL:R_0603
- added R37: 20K, Resistor_SMD_AKL:R_0603_1608Metric, symbol Resistor_US_AKL:R_0603
- added R38, R39, R40, R41, R42, R43: 150, Resistor_SMD_AKL:R_0603_1608Metric, symbol Resistor_US_AKL:R_0603
- added U15: MAX31856MUD+, EasyEDA:TSSOP-14_L5.0-W4.4-P0.65-LS6.4-BL, symbol EasyEDA:MAX31856MUD+
Connections:
- new net: C27.2, C29.1, R36.2, U15.4 (T+)
- new net: C27.1, C30.1, R35.2, U15.3 (T-)
- new net: R42.1, U15.13 (~{FAULT})
- new net: R38.1, U15.12 (SDI)
- new net: R40.1, U15.10 (SCK)
- new net: R39.1, U15.11 (SDO)
- new net: R37.2, U15.2 (BIAS)
- new net: R43.1, U15.7 (~{DRDY})
- new net: R41.1, U15.9 (~{CS})
- new net +3.3V: C28.1, C31.1, U15.5 (AVDD), U15.8 (DVDD)
- new net GND: C28.2, C29.2, C30.2, C31.2, U15.1 (AGND), U15.14 (DGND)
- new net SCK: R40.2
- new net SDI: R38.2
- new net SDO: R39.2
- new net TC+: R36.1
- new net TC-: R35.1, R37.1
- new net /CS: R41.2
- new net /DRDY: R43.2
- new net /FAULT: R42.2
