File: PLC4UNI NIZAO/PLC4UNI NIZAO/untitled.kicad_sch (KiCad schematic)
At the start: 1 part, among them U1 ESP32-S3-WROOM-1

Commit message: Commit 3
Parts:
- added C15, C16: 100NF, PCM_SparkFun-Capacitor:C_0603_1608Metric, symbol PCM_SparkFun-Capacitor:C
- added J5: Conn_02x07_Odd_Even, symbol Connector_Generic:Conn_02x07_Odd_Even
- added R25, R26: R_0603, symbol Device:R_US
- added R27: 22K, symbol Device:R_US
- added SW1: TS-1088-AR02016, symbol Switch:SW_DPST_x2
- added U2: ADS1115IDGS, Package_SO:TSSOP-10_3x3mm_P0.5mm, symbol Analog_ADC:ADS1115IDGS
Connections:
- net i2c_sda: now reaches U1.10 (IO17)
- net i2c_sda: now also J5.8 (Pin_8)
- net i2c_scl: now reaches U1.11 (IO18)
- net i2c_scl: now also J5.10 (Pin_10)
- net rs485_rx: now reaches U1.12 (IO8)
- net usb-: now reaches U1.13 (USB_D-)
- net usb-: now also J5.6 (Pin_6)
- net usb+: now reaches U1.14 (USB_D+)
- net usb+: now also J5.4 (Pin_4)
- net IN_NPN4: now reaches U1.15 (IO3)
- net OUT_PNP1: now reaches U1.16 (IO46)
- net rs485_tx: now reaches U1.17 (IO9)
- net rs485-com: now reaches U1.18 (IO10)
- net cs: now reaches U1.19 (IO11)
- net 3.3V: now reaches U1.2 (3V3)
- net 3.3V: now also J5.2 (Pin_2), R27.1
- net miso: now reaches U1.20 (IO12)
- net miso: now also J5.7 (Pin_7)
- net mosi: now reaches U1.21 (IO13)
- net mosi: now also J5.5 (Pin_5)
- net clk: now reaches U1.22 (IO14)
- net clk: now also J5.9 (Pin_9)
- net LED_INFO: now reaches U1.23 (IO21)
- net OUT_PNP2: now reaches U1.24 (IO47)
- net TEMP_CS: now reaches U1.25 (IO48)
- net OUT_RLY2: now reaches U1.26 (IO45)
- net IN_NPN1: now reaches U1.27 (IO0)
- net EN: now reaches U1.3 (EN)
- net EN: now also C16.1, R27.2, SW1.1 (A)
- net OUT_NPN1: now reaches U1.31 (IO38)
- net OUT_NPN2: now reaches U1.32 (IO39)
- net OUT_NPN3: now reaches U1.33 (IO40)
- net OUT_NPN4: now reaches U1.34 (IO41)
- net OUT_RLY1: now reaches U1.35 (IO42)
- net EMRX: now reaches U1.36 (RXD0)
- net EM_TX: now reaches U1.37 (TXD0)
- net IN_NPN3: now reaches U1.38 (IO2)
- net IN_NPN2: now reaches U1.39 (IO1)
- net IN_PNP1: now reaches U1.4 (IO4)
- net IN_PNP2: now reaches U1.5 (IO5)
- net IN_VDC_ADC: now reaches U1.6 (IO6)
- net acc_cs: now reaches U1.7 (IO7)
- net GPIO1: now reaches U1.8 (IO15)
- net GPIO1: now also J5.11 (Pin_11)
- net GPIO2: now reaches U1.9 (IO16)
- net GPIO2: now also J5.12 (Pin_12)
- new net +24V: R25.1
- new net +5V: J5.1 (Pin_1)
- new net CS: J5.3 (Pin_3)
- new net GND: C15.2, C16.2, J5.13 (Pin_13), J5.14 (Pin_14), R26.2, SW1.2 (B), U2.1 (ADDR), U2.3 (GND)
- new net IN-VDC-ADC: C15.1, R25.2, R26.1
- new net IN_0-10V/OUT3V: U2.6 (AIN2)
- new net IN_0-10V1/OUT3V: U2.7 (AIN3)
- new net IN_4-20_MA/OUT: U2.4 (AIN0)
- new net IN_4-20_MA1/OUT: U2.5 (AIN1)
- no-connect marks 0 -> 3
Other:
- added sheet EnergyMeterA1 (EnergyMeter.kicad_sch)
- added sheet IN-DI (IN-DI.kicad_sch)
- added sheet IN-DI1 (IN-DI.kicad_sch)
- added sheet IN-DI2 (IN-DI.kicad_sch)
- added sheet IN-DI3 (IN-DI.kicad_sch)
- added sheet IN_0-10V (IN-0-10V.kicad_sch)
- added sheet IN_0-10V1 (IN-0-10V.kicad_sch)
- added sheet IN_4-20_MA (4-20MA.kicad_sch)
- added sheet IN_4-20_MA1 (4-20MA.kicad_sch)
- added sheet RLY (RLY.kicad_sch)
- added sheet TC (TC.kicad_sch)
- moved on the sheet: U1

Commit message: commit 4 Schematic
Parts:
- added C17: 100NF, Capacitor_SMD_AKL:C_0603_1608Metric, symbol Capacitor_AKL:C_0603
- added LED5: LED_0603_Red, LED_SMD_AKL:LED_0603_1608Metric, symbol LED_AKL:LED_0603_Red
- added R50: 2.2K, Resistor_SMD_AKL:R_0603_1608Metric, symbol Resistor_US_AKL:R_0603
- added U9: RS485-PROTECT, MG_footprints:RS-485-PROTECT, symbol MG_CONNECTORS:RS485-PROTECT
Connections:
- net GND: now also U1.1 (GND), U1.40 (GND), U1.41 (GND), C17.2, LED5.1 (K), U9.2 (GND)
- net LED_INFO: now also R50.2
- net i2c_scl: now also U2.10 (SCL)
- net i2c_sda: now also U2.9 (SDA)
- net +3.3V: now reaches U2.8 (VDD)
- net +3.3V: now also C17.1, U9.1 (VCC)
- new net: LED5.2 (A), R50.1
- new net CON_RS485_A: U9.7 (A)
- new net CON_RS485_B: U9.8 (B)
- new net CON_RS485_G: U9.6 (RGND)
- new net RS485-CON: U9.5 (CON)
- new net RS485-RX: U9.4 (RXD)
- new net RS485-TX: U9.3 (TXD)
Other:
- added sheet IN-DI4 (IN-DI.kicad_sch)
- added sheet IN-DI5 (IN-DI.kicad_sch)
- added sheet OUT-0-10V (OUT-0-10V.kicad_sch)
- added sheet OUT-4-20MA (OUT-4-20MA.kicad_sch)
- added sheet OUT-NPN (OUT-NPN.kicad_sch)
- added sheet OUT-NPN1 (OUT-NPN.kicad_sch)
- added sheet OUT-NPN2 (OUT-NPN.kicad_sch)
- added sheet OUT-NPN3 (OUT-NPN.kicad_sch)
- added sheet OUT-PNP (OUT-PNP.kicad_sch)
- sheet EnergyMeterA1 ports: added CT_N, CT_P, RX, TX, VIN_N, VIN_P; removed none
- sheet TC ports: added SCK, SDI, SDO, TC+, TC-, /CS, /DRDY, /FAULT; removed none
- moved on the sheet: C15, C16, R25, R26, SW1A
